Commit message: Added dashbaord

File: src/social_nav_description/urdf/mir_social.urdf.xacro (robot description, xacro)
@@ -15,4 +15,7 @@
   <xacro:property name="wheel_len" value="0.032"/>
   <xacro:property name="wheel_sep" value="0.445208"/>
+  <!-- LiDAR range noise (Gaussian stddev, metres). Override via the SOCIAL_NAV_SCAN_NOISE env
+       var: 0.0 clean, 0.01 realistic (default), 0.03 stress. The demo scripts set it by profile. -->
+  <xacro:property name="scan_noise_stddev" value="$(optenv SOCIAL_NAV_SCAN_NOISE 0.01)"/>
   <material name="mir_white"><color rgba="0.9 0.9 0.92 1"/></material>
   <material name="mir_black"><color rgba="0.1 0.1 0.1 1"/></material>
@@ -131,4 +134,9 @@
         </scan>
         <range><min>0.20</min><max>12.0</max><resolution>0.01</resolution></range>
+        <noise>
+          <type>gaussian</type>
+          <mean>0.0</mean>
+          <stddev>${scan_noise_stddev}</stddev>
+        </noise>
       </ray>
       <plugin name="laser_plugin" filename="libgazebo_ros_ray_sensor.so">

Commit message: Trained

File: src/social_nav_description/urdf/mir_social.urdf.xacro (robot description, xacro)
@@ -61,7 +61,9 @@
     </joint>
     <link name="${name}_link">
+      <!-- Primitive cylinder visual (not the wheel.stl mesh): the mesh did not render as a wheel
+           in the GUI, and a cylinder is a faithful wheel shape that always shows in Gazebo + RViz. -->
       <visual>
-        <origin rpy="0 0 0" xyz="0 0 0"/>
-        <geometry><mesh filename="${mesh}/visual/wheel.stl"/></geometry>
+        <origin rpy="1.5707963 0 0" xyz="0 0 0"/>
+        <geometry><cylinder length="${wheel_len}" radius="${wheel_radius}"/></geometry>
         <material name="mir_black"/>
       </visual>
